File: AjoloteBoard.kicad_pcb (KiCad board)
At the start: 2 copper layers, 69 x 84.9 mm, 8 parts, among them SW1 On

Commit message: add heart logo
Parts:
- added svg2mod: G***, Aesthetics:heart, B.Cu at (158.8, 89.0)
Changed lines of the file:
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@@
-(kicad_pcb (version 20171130) (host pcbnew "(5.1.2)-1")
+(kicad_pcb (version 20171130) (host pcbnew "(5.1.4-0-10_14)")
   (general
     (thickness 1.6)
@@
     (tracks 90)
     (zones 0)
-    (modules 8)
+    (modules 9)
     (nets 5)
   )
@@
     (add_net "Net-(SW1-Pad1)")
   )
+  (module Aesthetics:heart (layer B.Cu)
+    (at 158.75 89.05 180)
+    (descr "Imported from heart.svg")
+    (tags svg2mod)
+    (attr smd)
+    (fp_text reference svg2mod (at 0 5.590896) (layer B.SilkS) hide
+      (effects (font (size 1.524 1.524) (thickness 0.3048)) (justify mirror))
+    )
+    (fp_text value G*** (at 0 -5.590896) (layer B.SilkS) hide
+      (effects (font (size 1.524 1.524) (thickness 0.3048)) (justify mirror))
+    )
+    (fp_poly (pts (xy -1.48108 2.324304) (xy -1.60345 2.318461) (xy -1.725158 2.300932) (xy -1.844992 2.271718)
+      (xy -1.96185 2.230818) (xy -2.07507 2.178452) (xy -2.183769 2.114291) (xy -2.287067 2.038444)
+      (xy -2.384301 1.95069) (xy -2.472275 1.853456) (xy -2.548123 1.750379) (xy -2.612394 1.641899)
+      (xy -2.66487 1.52879) (xy -2.70577 1.412153) (xy -2.735095 1.292649) (xy -2.752513 1.171382)
+      (xy -2.758356 1.049012) (xy -2.752513 0.926643) (xy -2.735095 0.805265) (xy -2.70588 0.685761)
+      (xy -2.66509 0.569124) (xy -2.612615 0.456125) (xy -2.548343 0.347646) (xy -2.472386 0.244348)
+      (xy -2.380884 0.143255) (xy 0.000035 -2.234356) (xy 2.380955 0.143255) (xy 2.472567 0.244459)
+      (xy 2.548414 0.347536) (xy 2.612465 0.456015) (xy 2.665051 0.569124) (xy 2.705841 0.685872)
+      (xy 2.735165 0.805375) (xy 2.752584 0.926643) (xy 2.758427 1.048902) (xy 2.752584 1.171272)
+      (xy 2.735055 1.292649) (xy 2.705731 1.412153) (xy 2.664941 1.5289) (xy 2.612465 1.641789)
+      (xy 2.548193 1.750379) (xy 2.472236 1.853456) (xy 2.384372 1.95058) (xy 2.287027 2.038444)
+      (xy 2.18373 2.114291) (xy 2.07503 2.178452) (xy 1.96181 2.230818) (xy 1.844953 2.271718)
+      (xy 1.725229 2.300932) (xy 1.603521 2.318461) (xy 1.481041 2.324304) (xy 1.35845 2.318461)
+      (xy 1.236852 2.300932) (xy 1.117128 2.271828) (xy 1.00016 2.231038) (xy 0.88683 2.178563)
+      (xy 0.778241 2.114511) (xy 0.674833 2.038664) (xy 0.57363 1.947383) (xy 0.15625 1.5289)
+      (xy 0.122081 1.500918) (xy 0.084184 1.480902) (xy 0.002157 1.464779) (xy -0.07994 1.48055)
+      (xy -0.117922 1.500404) (xy -0.15221 1.528239) (xy -0.573339 1.947052) (xy -0.674873 2.038664)
+      (xy -0.778281 2.114511) (xy -0.88698 2.178673) (xy -1.00009 2.231038) (xy -1.116947 2.271828)
+      (xy -1.236892 2.300932) (xy -1.35849 2.318461) (xy -1.48108 2.324304)) (layer B.Cu) (width 0))
+    (fp_poly (pts (xy 0 -2.542896) (xy -2.53909 -0.007352) (xy -2.641746 0.106128) (xy -2.730712 0.227037)
+      (xy -2.805987 0.354313) (xy -2.867572 0.486894) (xy -2.915467 0.623719) (xy -2.949671 0.763727)
+      (xy -2.970186 0.905855) (xy -2.97701 1.049043) (xy -2.970145 1.192229) (xy -2.94959 1.334351)
+      (xy -2.915346 1.474348) (xy -2.867413 1.611159) (xy -2.80579 1.743721) (xy -2.730479 1.870975)
+      (xy -2.641479 1.991857) (xy -2.53879 2.105306) (xy -2.425181 2.207848) (xy -2.30413 2.296721)
+      (xy -2.176698 2.371924) (xy -2.04395 2.433458) (xy -1.906947 2.481322) (xy -1.766754 2.515517)
+      (xy -1.624433 2.536042) (xy -1.481047 2.542896) (xy -1.337658 2.536081) (xy -1.195331 2.515595)
+      (xy -1.055128 2.481438) (xy -0.918112 2.43361) (xy -0.785346 2.372112) (xy -0.657893 2.296942)
+      (xy -0.536816 2.2081) (xy -0.423178 2.105588) (xy 0.001659 1.683002) (xy 0.423178 2.105588)
+      (xy 0.536816 2.2081) (xy 0.657893 2.296942) (xy 0.785346 2.372111) (xy 0.918112 2.43361)
+      (xy 1.055128 2.481437) (xy 1.195331 2.515594) (xy 1.337658 2.536079) (xy 1.481047 2.542894)
+      (xy 1.624433 2.536038) (xy 1.766754 2.515512) (xy 1.906948 2.481316) (xy 2.04395 2.43345)
+      (xy 2.176699 2.371914) (xy 2.304131 2.296708) (xy 2.425183 2.207833) (xy 2.538792 2.105288)
+      (xy 2.64148 1.991838) (xy 2.73048 1.870956) (xy 2.805791 1.743703) (xy 2.867413 1.61114)
+      (xy 2.915347 1.47433) (xy 2.94959 1.334333) (xy 2.970145 1.192211) (xy 2.97701 1.049025)
+      (xy 2.970186 0.905838) (xy 2.949672 0.76371) (xy 2.915467 0.623704) (xy 2.867573 0.486879)
+      (xy 2.805988 0.354299) (xy 2.730713 0.227025) (xy 2.641747 0.106118) (xy 2.539091 -0.007361)
+      (xy 0 -2.542896)) (layer B.Mask) (width 0.094249))
+  )
   (module footprints:Micro_interruptor_SPDT (layer B.Cu)

Commit message: silks led to back
Parts:
- D1, D2: moved to B.Cu
Changed lines of the file:
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@@
-(kicad_pcb (version 20171130) (host pcbnew "(5.1.4-0-10_14)")
+(kicad_pcb (version 20171130) (host pcbnew "(5.1.5-0-10_14)")
   (general
     (thickness 1.6)
@@
   (title_block
     (title "Axolote Board")
-    (date 2019-10-15)
-    (rev 0.3)
+    (date 2020-02-13)
+    (rev 1.1)
     (company "Electronic Cats")
     (comment 1 "Andrés Sabas")
@@
     (35 F.Paste user)
     (36 B.SilkS user)
-    (37 F.SilkS user hide)
+    (37 F.SilkS user)
     (38 B.Mask user)
-    (39 F.Mask user hide)
+    (39 F.Mask user)
     (40 Dwgs.User user)
     (41 Cmts.User user)
@@
     (pad "" np_thru_hole circle (at 1.35 -5.25 141) (size 0.9 0.9) (drill 0.7) (layers *.Cu *.Mask))
   )
-  (module LED_THT:LED_D5.0mm_Clear (layer F.Cu)
+  (module LED_THT:LED_D5.0mm_Clear (layer B.Cu)
     (at 180.82514 65)
     (descr "LED, diameter 5.0mm, 2 pins, http://cdn-reichelt.de/documents/datenblatt/A500/LL-504BC2E-009.pdf")
     (tags "LED diameter 5.0mm 2 pins")
-    (fp_text reference D2 (at 1.27 -3.96) (layer F.SilkS)
-      (effects (font (size 1 1) (thickness 0.15)))
-    )
-    (fp_text value LED (at 1.27 3.96) (layer F.Fab)
-      (effects (font (size 1 1) (thickness 0.15)))
-    )
-    (fp_arc (start 1.27 0) (end -1.29 1.54483) (angle -148.9) (layer F.SilkS) (width 0.12))
-    (fp_arc (start 1.27 0) (end -1.29 -1.54483) (angle 148.9) (layer F.SilkS) (width 0.12))
-    (fp_arc (start 1.27 0) (end -1.23 -1.469694) (angle 299.1) (layer F.Fab) (width 0.1))
-    (fp_circle (center 1.27 0) (end 3.77 0) (layer F.SilkS) (width 0.12))
-    (fp_circle (center 1.27 0) (end 3.77 0) (layer F.Fab) (width 0.1))
-    (fp_line (start 4.5 -3.25) (end -1.95 -3.25) (layer F.CrtYd) (width 0.05))
-    (fp_line (start 4.5 3.25) (end 4.5 -3.25) (layer F.CrtYd) (width 0.05))
-    (fp_line (start -1.95 3.25) (end 4.5 3.25) (layer F.CrtYd) (width 0.05))
-    (fp_line (start -1.95 -3.25) (end -1.95 3.25) (layer F.CrtYd) (width 0.05))
-    (fp_line (start -1.29 -1.545) (end -1.29 1.545) (layer F.SilkS) (width 0.12))
-    (fp_line (start -1.23 -1.469694) (end -1.23 1.469694) (layer F.Fab) (width 0.1))
-    (fp_text user %R (at 1.25 0) (layer F.Fab)
-      (effects (font (size 0.8 0.8) (thickness 0.2)))
-    )
+    (fp_text reference D2 (at 1.27 3.96) (layer B.SilkS)
+      (effects (font (size 1 1) (thickness 0.15)) (justify mirror))
+    )
+    (fp_text value LED (at 1.27 -3.96) (layer B.Fab)
+      (effects (font (size 1 1) (thickness 0.15)) (justify mirror))
+    )
+    (fp_text user %R (at 1.25 0) (layer B.Fab)
+      (effects (font (size 0.8 0.8) (thickness 0.2)) (justify mirror))
+    )
+    (fp_line (start -1.23 1.469694) (end -1.23 -1.469694) (layer B.Fab) (width 0.1))
+    (fp_line (start -1.29 1.545) (end -1.29 -1.545) (layer B.SilkS) (width 0.12))
+    (fp_line (start -1.95 3.25) (end -1.95 -3.25) (layer B.CrtYd) (width 0.05))
+    (fp_line (start -1.95 -3.25) (end 4.5 -3.25) (layer B.CrtYd) (width 0.05))
+    (fp_line (start 4.5 -3.25) (end 4.5 3.25) (layer B.CrtYd) (width 0.05))
+    (fp_line (start 4.5 3.25) (end -1.95 3.25) (layer B.CrtYd) (width 0.05))
+    (fp_circle (center 1.27 0) (end 3.77 0) (layer B.Fab) (width 0.1))
+    (fp_circle (center 1.27 0) (end 3.77 0) (layer B.SilkS) (width 0.12))
+    (fp_arc (start 1.27 0) (end -1.23 1.469694) (angle -299.1) (layer B.Fab) (width 0.1))
+    (fp_arc (start 1.27 0) (end -1.29 1.54483) (angle -148.9) (layer B.SilkS) (width 0.12))
+    (fp_arc (start 1.27 0) (end -1.29 -1.54483) (angle 148.9) (layer B.SilkS) (width 0.12))
+    (pad 1 thru_hole rect (at 0 0) (size 1.8 1.8) (drill 0.9) (layers *.Cu *.Mask)
+      (net 2 "Net-(D1-Pad1)"))
     (pad 2 thru_hole circle (at 2.54 0) (size 1.8 1.8) (drill 0.9) (layers *.Cu *.Mask)
       (net 1 "Net-(BT1-Pad1)"))
-    (pad 1 thru_hole rect (at 0 0) (size 1.8 1.8) (drill 0.9) (layers *.Cu *.Mask)
-      (net 2 "Net-(D1-Pad1)"))
     (model ${KISYS3DMOD}/LED_THT.3dshapes/LED_D5.0mm_Clear.wrl
       (at (xyz 0 0 0))
@@
     )
   )
-  (module LED_THT:LED_D5.0mm_Clear (layer F.Cu)
+  (module LED_THT:LED_D5.0mm_Clear (layer B.Cu)
     (at 134.68858 65)
     (descr "LED, diameter 5.0mm, 2 pins, http://cdn-reichelt.de/documents/datenblatt/A500/LL-504BC2E-009.pdf")
     (tags "LED diameter 5.0mm 2 pins")
-    (fp_text reference D1 (at 1.27 -3.96) (layer F.SilkS)
-      (effects (font (size 1 1) (thickness 0.15)))
-    )
-    (fp_text value LED (at 1.27 3.96) (layer F.Fab)
-      (effects (font (size 1 1) (thickness 0.15)))
-    )
-    (fp_arc (start 1.27 0) (end -1.29 1.54483) (angle -148.9) (layer F.SilkS) (width 0.12))
-    (fp_arc (start 1.27 0) (end -1.29 -1.54483) (angle 148.9) (layer F.SilkS) (width 0.12))
-    (fp_arc (start 1.27 0) (end -1.23 -1.469694) (angle 299.1) (layer F.Fab) (width 0.1))
-    (fp_circle (center 1.27 0) (end 3.77 0) (layer F.SilkS) (width 0.12))
-    (fp_circle (center 1.27 0) (end 3.77 0) (layer F.Fab) (width 0.1))
-    (fp_line (start 4.5 -3.25) (end -1.95 -3.25) (layer F.CrtYd) (width 0.05))
-    (fp_line (start 4.5 3.25) (end 4.5 -3.25) (layer F.CrtYd) (width 0.05))
-    (fp_line (start -1.95 3.25) (end 4.5 3.25) (layer F.CrtYd) (width 0.05))
-    (fp_line (start -1.95 -3.25) (end -1.95 3.25) (layer F.CrtYd) (width 0.05))
-    (fp_line (start -1.29 -1.545) (end -1.29 1.545) (layer F.SilkS) (width 0.12))
-    (fp_line (start -1.23 -1.469694) (end -1.23 1.469694) (layer F.Fab) (width 0.1))
-    (fp_text user %R (at 1.25 0) (layer F.Fab)
-      (effects (font (size 0.8 0.8) (thickness 0.2)))
+    (fp_text reference D1 (at 1.27 3.96) (layer B.SilkS)
+      (effects (font (size 1 1) (thickness 0.15)) (justify mirror))
+    )
+    (fp_text value LED (at 1.27 -3.96) (layer B.Fab)
+      (effects (font (size 1 1) (thickness 0.15)) (justify mirror))
+    )
+    (fp_arc (start 1.27 0) (end -1.29 -1.54483) (angle 148.9) (layer B.SilkS) (width 0.12))
+    (fp_arc (start 1.27 0) (end -1.29 1.54483) (angle -148.9) (layer B.SilkS) (width 0.12))
+    (fp_arc (start 1.27 0) (end -1.23 1.469694) (angle -299.1) (layer B.Fab) (width 0.1))
+    (fp_circle (center 1.27 0) (end 3.77 0) (layer B.SilkS) (width 0.12))
+    (fp_circle (center 1.27 0) (end 3.77 0) (layer B.Fab) (width 0.1))
+    (fp_line (start 4.5 3.25) (end -1.95 3.25) (layer B.CrtYd) (width 0.05))
+    (fp_line (start 4.5 -3.25) (end 4.5 3.25) (layer B.CrtYd) (width 0.05))
+    (fp_line (start -1.95 -3.25) (end 4.5 -3.25) (layer B.CrtYd) (width 0.05))
+    (fp_line (start -1.95 3.25) (end -1.95 -3.25) (layer B.CrtYd) (width 0.05))
+    (fp_line (start -1.29 1.545) (end -1.29 -1.545) (layer B.SilkS) (width 0.12))
+    (fp_line (start -1.23 1.469694) (end -1.23 -1.469694) (layer B.Fab) (width 0.1))
+    (fp_text user %R (at 1.25 0) (layer B.Fab)
+      (effects (font (size 0.8 0.8) (thickness 0.2)) (justify mirror))
     )
     (pad 2 thru_hole circle (at 2.54 0) (size 1.8 1.8) (drill 0.9) (layers *.Cu *.Mask)
@@
     (tags svg2mod)
     (attr smd)
-    (fp_text reference svg2mod (at 0 -45.573156) (layer F.SilkS) hide
+    (fp_text reference svg2mod (at -6.01 -35.04) (layer F.SilkS) hide
       (effects (font (size 1.524 1.524) (thickness 0.3048)))
     )
